File: TigardBR/0. Project/TigardBR.sch (EAGLE design)
At the start: 14 parts, among them SW1 DP4T, U1 FT2232HQ, U2 AP7366EA-33W5-7, U3 AP7366EA-18W5-7

Commit message: WIP
Parts:
- added C10, C12, C6, C8: 1uF, My-RLC:C_0603
- added C11, C13, C14, C15, C20, C21, C22, C23, C24, C25, C26, C27, C29, C5, C7, C9: 100nF, My-RLC:C_0603
- added C16, C17: 30pF, My-RLC:C_0603
- added C18, C19, C28, C30: 2.2uF, My-RLC:C_0603
- added FB2, FB3: 600R, 500mA, My-RLC:FB_0603
- added LED1, LED2: GREEN, My-LEDs:LED-0603-G
- added LED3: RED, My-LEDs:LED-0603-R
- added LED4, LED5: YELLOW, My-LEDs:LED-0603-Y
- added M1, M2: SSM3K335, My-Transistors:MOSFET-N-SSM3K335R
- added R10, R11, R14, R16, R18, R4, R5, R7, R8, R9: 10k, My-RLC:R_0603
- added R12: 2.2k, My-RLC:R_0603
- added R13: 12k, My-RLC:R_0603
- added R15, R17, R19, R20: 1k, My-RLC:R_0603
- added R2, R6: 1M, My-RLC:R_0603
- added RN1, RN5: 100k, My-RLC:RN_
- added RN2, RN4: 100R, My-RLC:RN_
- added SW2: DP4T-, My-Switches:DP4T-
- added U4, U5: SN74LVC8T245, My-ICs:SN74LVC8T245
- added U6: 93LC46BT-I/OT, My-ICs:93LC46BT-I/OT
- added Y1: 12MHz, My-Crystals:OSC-CHASSI-
- SW1: value DP4T -> DP4T-; device My-Switches:DP4T -> My-Switches:DP4T-
Connections:
- net N$1 renamed VBUS
- removed net VREF: SW1G$1.C
- new net !USB_READY: R17.1, R18.2, U1.!PWREN, U4.!OE, U5.!OE
- new net 1V8: C18.1, C19.1, C20.1, C21.1, C22.1, U1.VCORE, U1.VREGOUT
- new net AD0: RN1.9, RN5.9, U4.A8, U5.B8
- new net AD2: RN1.10, RN5.10, U4.A7, U5.B7
- new net AD4: RN1.11, RN5.11, U4.A6, U5.B6
- new net BD0: RN1.16, RN5.16, U4.A1, U5.B1
- new net BD1: RN1.15, RN5.15, U4.A2, U5.B2
- new net BD3: RN1.14, RN5.14, U4.A3, U5.B3
- new net BD4: RN1.13, RN5.13, U4.A4, U5.B4
- new net BD5: RN1.12, RN5.12, U4.A5, U5.B5
- new net N$1: LED2.A, R8.1
- new net N$10: RN4.11, U5.A6
- new net N$11: RN4.10, U5.A7
- new net N$12: RN2.1, U4.B1
- new net N$13: RN2.2, U4.B2
- new net N$14: RN2.3, U4.B3
- new net N$15: RN2.4, U4.B4
- new net N$16: RN2.5, U4.B5
- new net N$17: RN2.6, U4.B6
- new net N$18: RN2.7, U4.B7
- new net N$19: RN2.8, U4.B8
- new net N$2: R4.2, U4.DIR
- new net N$20: LED2.K, M1.D
- new net N$21: RN4.9, U5.A8
- new net N$22: R9.2, U1.EECS, U6.CS
- new net N$23: R10.2, U1.EECLK, U6.CLK
- new net N$24: R11.2, R12.2, U6.DO
- new net N$25: R12.1, U1.EEDATA, U6.DI
- new net N$26: LED1.A, R7.1
- new net N$27: C16.1, U1.OSCI, Y1.IN
- new net N$28: C17.1, U1.OSCO, Y1.OUT
- new net N$29: R13.1, U1.REF
- new net N$3: R5.1, U5.DIR
- new net N$30: R14.1, U1.!RESET
- new net N$31: C27.1, C28.1, FB2.2, U1.VPHY
- new net N$32: C29.1, C30.1, FB3.2, U1.VPLL
- new net N$33: M1.G, R15.2
- new net N$34: LED3.A, R16.1
- new net N$35: LED3.K, M2.D
- new net N$36: M2.G, R17.2
- new net N$37: LED4.A, R19.1
- new net N$38: LED4.K, U1.ACBUS3
- new net N$4: RN4.16, U5.A1
- new net N$41: LED5.K, U1.ACBUS4
- new net N$42: LED5.A, R20.1
- new net N$5: RN4.15, U5.A2
- new net N$6: RN4.14, U5.A3
- new net N$8: RN4.13, U5.A4
- new net N$9: RN4.12, U5.A5
- new net VLOGIC: C10.1, C5.1, C6.1, C9.1, R2.2, RN5.1, RN5.2, RN5.3, RN5.4, RN5.5, RN5.6, RN5.7, RN5.8, SW1G$1.C, U4.VCCB, U5.VCCB
- net 0V: now also C10.2, C11.2, C12.2, C13.2, C14.2, C15.2, C16.2, C17.2, C18.2, C19.2, C20.2, C21.2, C22.2, C23.2, C24.2, C25.2, C26.2, C27.2, C28.2, C29.2, C30.2, C5.2, C6.2, C7.2, C8.2, C9.2, LED1.K, M1.S, M2.S, R13.2, R2.1, R5.2, R6.1, U1.AGND, U1.GND, U1.TEST, U4.GND, U5.GND, U6.GND, Y1.CH
- net 1.8V: now also C14.1, SW2G$1.NO2
- net 3.3V: now also C11.1, C12.1, C13.1, C15.1, C23.1, C24.1, C25.1, C26.1, C7.1, C8.1, FB2.1, FB3.1, R10.1, R11.1, R14.2, R18.1, R19.2, R20.2, R4.1, R9.1, RN1.1, RN1.2, RN1.3, RN1.4, RN1.5, RN1.6, RN1.7, RN1.8, SW2G$1.NO1, U1.VCCIO, U1.VREGIN, U4.VCCA, U5.VCCA, U6.VDD
- net 5.0V: now also R16.2, R7.2, R8.2, SW2G$1.NC
- net USB_D+: now also U1.DP
- net USB_D-: now also U1.DM
- net VTARGET: now also R15.1, R6.2, SW2G$1.C
Other:
- note added: "*"
- note added: "* The switches are break-before-make (BBM, non-shorting type)."
- note added: "Many configurations are possible: - The target can be powered either externally or by the TigardBR. - The LOGIC levels may be the same as or different from the target SUPPLY voltage. - The LOGIC levels can be set either by the TigardBR or by the target’s own EXTERNAL power supply."
- note added: "external power ("target self-powered")"
- note added: "same as target supply"
- moved on the sheet: C1, C2, C3, C4, CN1, D1, FB1, R1, R3, RT1, SW1, U2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

Commit message: WIP
Parts:
- added R21: 2.2k, My-RLC:R_0603
- LED2: value GREEN -> BLUE; device My-LEDs:LED-0603-G -> My-LEDs:LED-0603-B
- R15, R17, R19, R20: value 1k -> 4k7
- R16, R7, R8: value 10k -> 4k7
Connections:
- new net AD1: RN4.1, U1.ADBUS1
- new net AD3: RN4.2, U1.ADBUS3
- new net AD5: RN4.3, U1.ADBUS5
- new net AD6: RN4.4, U1.ADBUS6
- new net BD2: RN4.5, U1.BDBUS2
- new net BD6: RN4.6, U1.BDBUS6
- new net BD7: R21.2, U1.BDBUS7
- net 3.3V: now also R16.2, R7.2, R8.2
- net 5.0V: no longer R16.2, R7.2, R8.2
- net AD0: now also U1.ADBUS0
- net AD2: now also U1.ADBUS2
- net AD4: now also U1.ADBUS4
- net BD0: now also U1.BDBUS0
- net BD1: now also U1.BDBUS1
- net BD3: now also U1.BDBUS3
- net BD4: now also U1.BDBUS4
- net BD5: now also R21.1, U1.BDBUS5
Other:
- moved on the sheet: C1, C11, C12, C13, C14, C15, C16, C17, C18, C19, C2, C20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
