File: TigardBR/0. Project/TigardBR.sch (EAGLE design)
At the start: 77 parts, among them M1 SSM3K335, M2 SSM3K335, SW1 DP4T-, SW2 DP4T-, U1 FT2232HQ, U2 AP7366EA-33W5-7, U3 AP7366EA-18W5-7, U4 SN74LVC8T245, U5 SN74LVC8T245, U6 93LC46BT-I/OT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

Commit message: WIP
Parts:
- added CN2: JTAG/SWD, My-Connectors:JTAG
- added CN3: I2C, My-PinHeaders:PINHD-1X04_2.54
- added JP1: JTAG, My-PinHeaders:PINHD-1X09_2.54
- added JP2: SPI, My-PinHeaders:PINHD-2X04_2.54
- added JP3: UART, My-PinHeaders:PINHD-1X09_2.54
- added JP4: LOGIC ANALYSER, My-PinHeaders:PINHD-2X07_2.54
- added R22: 330R, My-RLC:R_0603
- added R23: 0R, My-RLC:R_0603
- added R24, R25: 10k, My-RLC:R_0603
- added SJ1: 2P-NO, My-Jumpers:2P-NO
- added SW3: DP2T-STRAIGHT-SMD, My-Switches:DP2T-STRAIGHT-SMD
Connections:
- new net AD0_EXT: JP3.3, JP4.7, RN2.9
- new net AD1_EXT: JP3.4, JP4.8, R23.1, RN5.16, U5.B1
- new net AD2_EXT: JP3.5, RN2.10
- new net AD3_EXT: JP3.6, RN5.15, U5.B2
- new net AD4_EXT: JP3.7, RN2.11
- new net AD5_EXT: JP3.8, RN5.14, U5.B3
- new net AD6_EXT: JP3.9, RN5.13, U5.B4
- new net BD0_EXT: CN2.TCK, CN3.4, JP1.3, JP2.6, JP4.1, RN2.16
- new net BD1_EXT: CN2.TDI, CN3.3, JP1.4, JP2.8, JP4.2, R22.2, RN2.15, SJ1.3
- new net BD2_EXT: JP4.3, RN5.12, SW3SW2.C, U5.B5
- new net BD2_EXT_SWITCHED: CN2.TDO, JP1.5, JP2.3, SW3SW2.NC
- new net BD3_EXT: JP1.6, JP2.1, JP4.4, RN2.14, SW3SW1.NC
- new net BD4_EXT: JP1.7, JP4.5, RN2.13
- new net BD5_EXT: CN2.!RST, JP1.8, JP4.6, RN2.12
- new net BD6_EXT: JP1.9, R23.2, RN5.11, U5.B6
- new net N$43: CN2.TMS, SW3SW1.C
- new net N$44: JP2.4, R24.1
- new net N$45: JP2.5, R25.1
- new net SWDIO: R22.1, SJ1.1, SW3SW1.NO, SW3SW2.NO
- net 0V: now also CN2.GND, CN2.GND2, CN2.GND3, CN3.1, JP1.2, JP2.7, JP3.2, JP4.10, JP4.9
- net AD4: no longer RN5.11, U5.B6
- net BD0: no longer RN5.16, U5.B1
- net BD1: no longer RN5.15, U5.B2
- net BD3: no longer RN5.14, U5.B3
- net BD4: no longer RN5.13, U5.B4
- net BD5: no longer RN5.12, U5.B5
- net VTARGET: now also CN2.VDD, CN3.2, JP1.1, JP2.2, JP3.1, R24.2, R25.2
Other:
- note added: "!SRST"
- note added: "!TRST"
- note added: "!UART_CTS"
- note added: "!UART_DCD"
- note added: "!UART_DSR"
- note added: "!UART_DTR"
- note added: "!UART_RTS"
- note added: "CLK"
- note added: "CS"
- note added: "ICE_CDONE"
- note added: "MISO"
- note added: "MOSI"
- note added: "SCL"
- note added: "SDA"
- note added: "SWD and JTAG support"
- note added: "SWDIO"
- note added: "TCK"
- note added: "TDI"
- note added: "TDO"
- note added: "TMS"
- note added: "UART_RX"
- note added: "UART_TX"
- note added: "xPB0"
- note added: "xPB1"
- note added: "xPB2"
- note added: "xPB3"
- note added: "xPB4"
- note added: "xPB5"
- note added: "xPB6"
- note added: "xPB7"

Commit message: WIP
Parts:
- added JP5: SPI, My-PinHeaders:PINHD-2X03_2.54
Connections:
- net BD7 renamed BDBUS7
- removed net AD0_EXT: JP3.3, JP4.7, RN2.9
- removed net AD1_EXT: JP3.4, JP4.8, R23.1, RN5.16, U5.B1
- removed net AD2_EXT: JP3.5, RN2.10
- removed net AD3_EXT: JP3.6, RN5.15, U5.B2
- removed net AD4_EXT: JP3.7, RN2.11
- removed net AD5_EXT: JP3.8, RN5.14, U5.B3
- removed net AD6_EXT: JP3.9, RN5.13, U5.B4
- removed net BD0_EXT: CN2.TCK, CN3.4, JP1.3, JP2.6, JP4.1, RN2.16
- removed net BD1_EXT: CN2.TDI, CN3.3, JP1.4, JP2.8, JP4.2, R22.2, RN2.15, SJ1.3
- removed net BD2_EXT: JP4.3, RN5.12, SW3SW2.C, U5.B5
- removed net BD3_EXT: JP1.6, JP2.1, JP4.4, RN2.14, SW3SW1.NC
- removed net BD4_EXT: JP1.7, JP4.5, RN2.13
- removed net BD5_EXT: CN2.!RST, JP1.8, JP4.6, RN2.12
- removed net BD6_EXT: JP1.9, R23.2, RN5.11, U5.B6
- new net ADBUS0: RN1.9, RN5.9, U1.ADBUS0, U4.A8, U5.B8
- new net ADBUS1: RN4.1, U1.ADBUS1
- new net ADBUS2: RN1.10, RN5.10, U1.ADBUS2, U4.A7, U5.B7
- new net ADBUS3: RN4.2, U1.ADBUS3
- new net ADBUS4: RN1.11, U1.ADBUS4, U4.A6
- new net ADBUS5: RN4.3, U1.ADBUS5
- new net ADBUS6: RN4.4, U1.ADBUS6
- new net ADBUS7: U1.ADBUS7
- new net BDBUS0: RN1.16, U1.BDBUS0, U4.A1
- new net BDBUS1: RN1.15, U1.BDBUS1, U4.A2
- new net BDBUS2: RN4.5, U1.BDBUS2
- new net BDBUS3: RN1.14, U1.BDBUS3, U4.A3
- new net BDBUS4: RN1.13, U1.BDBUS4, U4.A4
- new net BDBUS5: R21.1, RN1.12, U1.BDBUS5, U4.A5
- new net BDBUS6: RN4.6, U1.BDBUS6
- net AD0: now also JP3.3, JP4.7, RN2.9; no longer RN1.9, RN5.9, U1.ADBUS0, U4.A8, U5.B8
- net AD1: now also JP3.4, JP4.8, R23.1, RN5.16, U5.B1; no longer RN4.1, U1.ADBUS1
- net AD2: now also JP3.5, RN2.10; no longer RN1.10, RN5.10, U1.ADBUS2, U4.A7, U5.B7
- net AD3: now also JP3.6, RN5.15, U5.B2; no longer RN4.2, U1.ADBUS3
- net AD4: now also JP3.7, RN2.11; no longer RN1.11, U1.ADBUS4, U4.A6
- net AD5: now also JP3.8, RN5.14, U5.B3; no longer RN4.3, U1.ADBUS5
- net AD6: now also JP3.9, RN5.13, U5.B4; no longer RN4.4, U1.ADBUS6
- net BD0: now also CN2.TCK, CN3.4, JP1.3, JP2.6, JP4.1, JP5.3, RN2.16; no longer RN1.16, U1.BDBUS0, U4.A1
- net BD1: now also CN2.TDI, CN3.3, JP1.4, JP2.8, JP4.2, R22.2, RN2.15, SJ1.3; no longer RN1.15, U1.BDBUS1, U4.A2
- net BD2: now also JP4.3, RN5.12, SW3SW2.C, U5.B5; no longer RN4.5, U1.BDBUS2
- net BD2_EXT_SWITCHED: now also JP5.1
- net BD3: now also JP1.6, JP2.1, JP4.4, RN2.14, SW3SW1.NC; no longer RN1.14, U1.BDBUS3, U4.A3
- net BD4: now also JP1.7, JP4.5, RN2.13; no longer RN1.13, U1.BDBUS4, U4.A4
- net BD5: now also CN2.!RST, JP1.8, JP4.6, JP5.5, RN2.12; no longer R21.1, RN1.12, U1.BDBUS5, U4.A5
- net BD6: now also JP1.9, R23.2, RN5.11, U5.B6; no longer RN4.6, U1.BDBUS6
Other:
- note added: "!CS"
- note added: "!HOLD!/!RESET!"
- note added: "!WP"
- note added: "SCLK"
- note added: "TCK | SWDCLK"
- note added: "TDO | SWO"
- note added: "TMS | SWDIO"
- note removed: "CLK"
- note removed: "CS"
- moved on the sheet: R22, RN4, SJ1, SW3

Commit message: WIP
Parts:
- added Q3, Q4: NPN-PMMT491, My-Transistors:NPN-PMMT491
- added R26, R27: 4k7 (5%), My-RLC:R_0402
- added R28, R29: 0R, My-RLC:R_0603
Connections:
- new net ESP_EN: Q3.C
- new net ESP_IO0: Q4.C
- new net ESP_RX: R28.2
- new net ESP_TX: R29.2
- new net N$46: Q3.B, R26.1
- new net N$47: Q4.B, R27.1
- new net N$48: R28.1
- new net N$49: R29.1
- new net USB_DTR: Q4.E, R26.2
- new net USB_RTS: Q3.E, R27.2
Other:
- moved on the sheet: C10, C11, C12, C5, C6, C7, C8, C9, CN2, R21, R22, R23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

Commit message: WIP
Parts:
- added C31, C32: 1nF, My-RLC:C_0603
- added JP6: ESP32 UART, My-PinHeaders:PINHD-2X03_2.54
- added R30, R31: 10k, My-RLC:R_0603
- R26, R27: value 4k7 (5%) -> 10k; device My-RLC:R_0402 -> My-RLC:R_0603; PN ERJ-2GEJ472X -> (none)
Connections:
- removed net N$48: R28.1
- removed net N$49: R29.1
- removed net USB_DTR: Q4.E, R26.2
- removed net USB_RTS: Q3.E, R27.2
- net 0V: now also C31.2, C32.2, JP6.4
- net AD0: now also R29.1
- net AD1: now also R28.1
- net AD2: now also Q3.E, R27.1
- net AD4: now also Q4.E, R26.1
- net ESP_EN: now also C31.1, JP6.1, R30.1
- net ESP_IO0: now also C32.1, JP6.6, R31.1
- net ESP_RX: now also JP6.5, R29.2; no longer R28.2
- net ESP_TX: now also JP6.3, R28.2; no longer R29.2
- net N$46: now also R26.2; no longer R26.1
- net N$47: now also R27.2; no longer R27.1
- net VTARGET: now also JP6.2, R30.2, R31.2
Other:
- note added: "With automatic download and run functionality."
- moved on the sheet: Q3, Q4, R26, R27, R28, R29

Commit message: WIP
Parts:
- added C33: 100nF, My-RLC:C_0603
- added C34: 10uF, My-RLC:CP_1206_POL
- added C35: 1uF, My-RLC:C_0603
- added D2, D4, D6: SDT5A50, My-Diodes:SCHOTTKY-SDT5A50SA
- added M6: SSM3J332, My-Transistors:MOSFET-P-SSM3J332R
- added R32, R33, R34: 10k, My-RLC:R_0603
- added U7: TLV1117LV, My-LDOs:1117-3.3V
- added U8: SN74AHC125, My-ICs:QUAD-BUFFER-
- C1: value 100nF -> 10uF; device My-RLC:C_0603 -> My-RLC:CP_1206_POL; PN (none) -> T494A106M016AT
- C13, C14: PN (none) -> CL10B104JB8NNNC
- C2: value 2.2uF -> 10uF; device My-RLC:C_0603 -> My-RLC:CP_1206_POL; PN (none) -> T494A106M016AT
- C3: value 2.2uF -> 100nF; PN (none) -> CL10B104JB8NNNC
- C4: value 2.2uF -> 1uF; PN (none) -> CL10B104JB8NNNC
- Q3, Q4: value NPN-PMMT491 -> PMMT491; device My-Transistors:NPN-PMMT491 -> My-Transistors:BJT-N-PMMT491
- U2: value AP7366EA-33W5-7 -> TLV1117LV; device My-LDOs:AP7366EA-33W5-7 -> My-LDOs:1117-3.3V; PN (none) -> TLV1117LV18DCYR
- U3: value AP7366EA-18W5-7 -> 74LVC1G04; device My-LDOs:AP7366EA-18W5-7 -> My-ICs:SINGLE-INVERTER-74LVC1G04GV
Connections:
- new net ESP_TCK: U8-D.Y
- new net ESP_TDI: U8-C.Y
- new net ESP_TDO: U8-B.A
- new net ESP_TMS: U8-A.Y
- new net N$48: D1.VCC, D4.A, R34.2, R7.2, RT1.1
- new net N$49: C4.2, D6.K, M6.G, R32.2
- new net N$50: C33.1, M6.D, U3G$2.VDD, U8G$5.VDD
- new net N$51: D2.A, R33.1, U3-A.Y
- new net N$52: C35.1, D2.K, R33.2, U8-A.!OE
- net 0V: now also C1.-, C2.-, C33.2, C34.-, C35.2, D6.A, R32.1, R34.1, U3G$2.VSS, U7.GND, U8G$5.VSS; no longer C1.2, C2.2, C4.2, U3.GND
- net 1.8V: now also C34.+, U2.OUT; no longer C4.1, U3.OUT
- net 3.3V: now also C1.+, U2.IN, U7.OUT; no longer C3.1, R7.2, U2.OUT, U3.EN, U3.IN
- net 5.0V: now also C2.+, C3.1, U7.IN; no longer C1.1, C2.1, U2.EN, U2.IN
- net BD0: now also U8-D.A
- net BD1: now also U8-C.A
- net BD2_EXT_SWITCHED: now also U8-B.Y
- net BD3: now also U8-A.A
- net ESP_EN: now also U3-A.A
- net N$7: now also D4.K; no longer D1.VCC, RT1.1
- net VTARGET: now also C4.1, M6.S
Other:
- moved on the sheet: C13, C14, C3, C31, C32, C4, CN1, D1, FB1, LED1, R1, R3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

Commit message: WIP
Connections:
- removed net N$52: C35.1, D2.K, R33.2, U8-A.!OE
- new net !ESP_EN: C35.1, D2.K, R33.2, U8-A.!OE, U8-B.!OE, U8-C.!OE, U8-D.!OE
Other:
- note added: "FTDI"
- note added: "TARGET"
- moved on the sheet: C33, C35, D2, D6, R32, R33, U3-A, U8-A, U8-B, U8-C, U8-D

Commit message: WIP
Parts:
- removed JP6: ESP32 UART, My-PinHeaders:PINHD-2X03_2.54
- added CN4: 1.27mm, My-Connectors:JTAG
- added CN5: 2.54mm, My-PinHeaders:PINHD-2X05_2.54
- added CN6: 2.54mm, My-PinHeaders:PINHD-2X03_2.54
- CN2: PN (none) -> 20021121-00010C4LF
- R30, R31: value 10k -> DNP
Connections:
- net 0V: now also CN4.GND, CN4.GND2, CN4.GND3, CN5.3, CN5.5, CN5.9, CN6.4; no longer JP6.4
- net ESP_EN: now also CN6.1; no longer JP6.1
- net ESP_IO0: now also CN6.6; no longer JP6.6
- net ESP_RX: now also CN6.5; no longer JP6.5
- net ESP_TCK: now also CN4.TCK, CN5.4
- net ESP_TDI: now also CN4.TDI, CN5.8
- net ESP_TDO: now also CN4.TDO, CN5.6
- net ESP_TMS: now also CN4.TMS, CN5.2
- net ESP_TX: now also CN6.3; no longer JP6.3
- net VLOGIC: now also C4.1, M6.S, R30.2, R31.2
- net VTARGET: now also CN4.VDD, CN5.1, CN6.2; no longer C4.1, JP6.2, M6.S, R30.2, R31.2
Other:
- note added: "* From ESP-IDF Programing Guide: "The JTAG port on the ESP32 is an industry-standard JTAG port which lacks (and does not need) the TRST pin.""
- note added: "Delay circuit to protect the ESP32 from JTAG interference during power-up or reset."
- note added: "FTDI SIDE"
- note added: "TARGET SIDE"
- note removed: "FTDI"
- note removed: "TARGET"
- moved on the sheet: C33, C35, C4, D2, D6, M6, R32, R33, U3-A, U8-A, U8-B, U8-C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
